File: USB_HUB.brd (EAGLE design)
At the start: 76.2 x 38 mm, 69 parts, among them U1 TLV71211DBVR, U2 LP5907MFX-3.3/NOPB

Commit message: Fixed
Parts:
- removed C13, C5, C6, C7: 0.1uF, SparkFun-Capacitors:0603
- removed R10, R11, R21, R9: 0, SparkFun-Resistors:0805
- removed USB1_+5V, USB1_DM, USB1_DP, USB1_GND, USB2_+5V, USB2_DM, USB2_DP, USB2_GND, USB3_+5V, USB3_DM, USB3_DP, USB3_GND, USB4_+5V, USB4_DM, USB4_DP, USB4_GND: (no value), SparkFun-Connectors:1X01
- added C19, C20, C25, C29: 0.1uF, SparkFun-Capacitors:0603
- added R17, R18, R19, R20: 0, SparkFun-Resistors:0805
- added U$11, U$2, U$3, U$4: T2I5P, BackplaneParts:T2I5P
- moved C2 17.4 mm to (72.6, 15.7)
- moved C3 17.4 mm to (72.6, 20.8)
- moved R5 17.4 mm to (60.5, 18.3)
- moved Y2 17.4 mm to (67.6, 18.3)
- moved R12 11.7 mm to (17.0, 24.4), turned to 270 degrees
- moved C15 4.64 mm to (39.1, 8.38)
- moved C16 3.05 mm to (33.8, 6.86)
- moved C8 3.05 mm to (36.1, 6.86)
- moved R3 0.25 mm to (44.5, 9.65)
Connections:
- removed net N$12: C13.1, R21.1, USB1_+5V.1
- removed net N$13: C5.1, R9.1, USB2_+5V.1
- removed net N$14: C6.1, R10.1, USB3_+5V.1
- removed net N$15: C7.1, R11.1, USB4_+5V.1
- new net USB1_+5V: C19.1, R17.1, U$11.P$6
- new net USB2_+5V: C20.1, R18.1, U$2.P$6
- new net USB3_+5V: C25.1, R19.1, U$3.P$6
- new net USB4_+5V: C29.1, R20.1, U$4.P$6
- net +5V: now also R17.2, R18.2, R19.2, R20.2; no longer R10.2, R11.2, R21.2, R9.2
- net DM1: now also U$11.P$5; no longer USB1_DM.1
- net DM2: now also U$2.P$5; no longer USB2_DM.1
- net DM3: now also U$3.P$5; no longer USB3_DM.1
- net DM4: now also U$4.P$5; no longer USB4_DM.1
- net DP1: now also U$11.P$4; no longer USB1_DP.1
- net DP2: now also U$2.P$4; no longer USB2_DP.1
- net DP3: now also U$3.P$4; no longer USB3_DP.1
- net DP4: now also U$4.P$4; no longer USB4_DP.1
- net GND: now also C19.2, C20.2, C25.2, C29.2, U$11.P$3, U$2.P$3, U$3.P$3, U$4.P$3; no longer C13.2, C5.2, C6.2, C7.2, USB1_GND.1, USB2_GND.1, USB3_GND.1, USB4_GND.1
Routing:
- net DP1: track 29.9 -> 57.9 mm
- net N$5: track 24.7 -> 45.2 mm, vias 0 -> 2
- net N$6: track 25.2 -> 45.6 mm, vias 0 -> 2
- net DM1: track 25.2 -> 40.0 mm
- net +5V: track 64.9 -> 75.8 mm, vias 0 -> 2
- net PWRCTL4/BATEN4: track 11.9 -> 22.5 mm, vias 0 -> 2
- net USB2_+5V: track 0.00 -> 10.6 mm
- net USB3_+5V: track 0.00 -> 10.6 mm
- net VDD: track 99.1 -> 89.4 mm
- net DM4: track 29.0 -> 20.0 mm, vias 1 -> 2
- net USB1_+5V: track 0.00 -> 8.31 mm
- net USB4_+5V: track 0.00 -> 7.95 mm
- net 3.3V: track 36.9 -> 29.3 mm, vias 2 -> 4
- net N$15: track 6.10 -> 0.00 mm
- net N$14: track 5.90 -> 0.00 mm
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
Commit message: this should work..
Parts:
- moved R18 30.9 mm to (57.9, 27.7), turned to 90 degrees
- moved U$2 30.7 mm to (66.0, 28.2), turned to 90 degrees
- moved C20 25.1 mm to (57.9, 23.6), turned to 270 degrees
- moved C2 20.4 mm to (56.6, 3.05), turned to 270 degrees
- moved C3 19.2 mm to (56.6, 10.2), turned to 90 degrees
- moved R5 19.2 mm to (45.2, 6.60)
- moved Y2 19.2 mm to (52.3, 6.60)
- moved U$4 18.4 mm to (14.7, 36.6), turned to 180 degrees
- moved C29 2.03 mm to (37.1, 32.8)
- moved R20 2.03 mm to (36.3, 35.3)
- moved C23 1.61 mm to (37.3, 28.2)
- moved C24 1.61 mm to (34.8, 28.2)
- moved C11 1.48 mm to (45.7, 12.7)
- moved R3 1.27 mm to (45.7, 9.65)
- moved C12 1.05 mm to (40.9, 29.5)
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Routing:
- net N$5: track 45.2 -> 23.6 mm, vias 2 -> 0
- net N$6: track 45.6 -> 24.0 mm, vias 2 -> 0
- net DP1: track 57.9 -> 40.8 mm
- net +5V: track 75.8 -> 89.0 mm
- net GND: track 44.6 -> 32.5 mm, vias 10 -> 8
- net USB4_+5V: track 7.95 -> 20.0 mm
- net DM4: track 20.0 -> 25.8 mm
- net DP_UP: track 45.8 -> 51.4 mm
- net USB2_+5V: track 10.6 -> 7.15 mm
- net DP4: track 22.1 -> 25.6 mm, vias 1 -> 2
- net DP2: track 23.0 -> 19.9 mm, vias 3 -> 1
- net USB3_+5V: track 10.6 -> 7.62 mm
- net DM2: track 22.8 -> 20.1 mm
- net DP3: track 15.8 -> 13.8 mm, vias 0 -> 1
- net N$2: track 4.98 -> 6.25 mm
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