File: USB_HUB.sch (EAGLE design)
At the start: 69 parts, among them U1 TLV71211DBVR, U2 LP5907MFX-3.3/NOPB

Commit message: Fixed
Parts:
- removed C13, C5, C6, C7: 0.1uF, SparkFun-Capacitors:0.1UF-0603-25V-(+80/-20%)
- removed R10, R11, R21, R9: 0, SparkFun-Resistors:RESISTOR0805
- removed USB1_+5V, USB1_DM, USB1_DP, USB1_GND, USB2_+5V, USB2_DM, USB2_DP, USB2_GND, USB3_+5V, USB3_DM, USB3_DP, USB3_GND, USB4_+5V, USB4_DM, USB4_DP, USB4_GND: (no value), SparkFun-Connectors:M01PTH
- added C19, C20, C25, C29: 0.1uF, SparkFun-Capacitors:0.1UF-0603-25V-(+80/-20%)
- added R17, R18, R19, R20: 0, SparkFun-Resistors:RESISTOR0805
- added U$11, U$2, U$3, U$4: T2I5P, BackplaneParts:T2I5P
Connections:
- removed net N$12: C13.1, R21.1, USB1_+5V.1
- removed net N$13: C5.1, R9.1, USB2_+5V.1
- removed net N$14: C6.1, R10.1, USB3_+5V.1
- removed net N$15: C7.1, R11.1, USB4_+5V.1
- new net USB1_+5V: C19.1, R17.1, U$11.5
- new net USB2_+5V: C20.1, R18.1, U$2.5
- new net USB3_+5V: C25.1, R19.1, U$3.5
- new net USB4_+5V: C29.1, R20.1, U$4.5
- net +5V: now also R17.2, R18.2, R19.2, R20.2; no longer R10.2, R11.2, R21.2, R9.2
- net DM1: now also U$11.4; no longer USB1_DM.1
- net DM2: now also U$2.4; no longer USB2_DM.1
- net DM3: now also U$3.4; no longer USB3_DM.1
- net DM4: now also U$4.4; no longer USB4_DM.1
- net DP1: now also U$11.3; no longer USB1_DP.1
- net DP2: now also U$2.3; no longer USB2_DP.1
- net DP3: now also U$3.3; no longer USB3_DP.1
- net DP4: now also U$4.3; no longer USB4_DP.1
- net GND: now also C19.2, C20.2, C25.2, C29.2, U$11.2, U$2.2, U$3.2, U$4.2; no longer C13.2, C5.2, C6.2, C7.2, USB1_GND.1, USB2_GND.1, USB3_GND.1, USB4_GND.1
